Commit message: file rename for msg fix

File: neato/urdf/neato.urdf.xacro (robot description, xacro)
@@ -6,5 +6,5 @@
             <origin xyz="0.150 -0.165 -0.040" rpy="0 0 1.57" />
             <geometry>
-                <mesh filename="package://neato_node/meshes/neato.dae" scale="0.025 0.025 0.025" />
+                <mesh filename="package://neato/meshes/neato.dae" scale="0.025 0.025 0.025" />
             </geometry>
         </visual>
@@ -13,5 +13,5 @@
         <origin xyz="0 0 0" rpy="0 0 0" />
         <geometry>
-          <mesh filename="package://neato_node/meshes/neato.stl"/>
+          <mesh filename="package://neato/meshes/neato.stl"/>
         </geometry>
       </collision>
